Commit message: Integration of LiDAR plugin into main package with minor updates
Deletion of the velodyne package

File: qutms_autonomous/urdf/qev2_base_gazebo.xacro (robot description, xacro)
@@ -35,5 +35,5 @@
 	  </xacro:qev2_horizon_lidar>
   </xacro:if>
-  <!-- Add Horizon LIDAR using the Velodyne package -->
+  <!-- Add Cameras -->
   <xacro:if value="$(arg camera_enabled)">
     <xacro:qev2_zed_camera parent="base_link">

File: qutms_autonomous/urdf/sensors/qev2_horizon_lidar.urdf.xacro (robot description, xacro)
@@ -1,4 +1,4 @@
 <?xml version="1.0"?>
-<robot xmlns:xacro="http://ros.org/wiki/xacro" name="VLP-16">
+<robot xmlns:xacro="http://ros.org/wiki/xacro" name="Horizon">
   <xacro:property name="M_PI" value="3.1415926535897931" />
   <xacro:macro name="qev2_horizon_lidar" params=" *origin
@@ -8,7 +8,7 @@
       <xacro:insert_block name="origin" />
       <parent link="${parent}"/>
-      <child link="${name}"/>
+      <child link="${name}_base_link"/>
     </joint>
-    <link name="${name}">
+    <link name="${name}_base_link">
       <inertial>
         <mass value="1.18"/>
@@ -28,14 +28,13 @@
       </collision>
     </link>
-    <!-- Gazebo requires the velodyne_gazebo_plugins package -->
-    <gazebo reference="${name}">
+    <gazebo reference="${name}_base_link">
       <sensor type="ray" name="${name}_sensor">
         <pose>0 0 0 0 0 0</pose>
+        <update_rate>30.0</update_rate>
         <visualize>false</visualize>
-        <update_rate>30</update_rate>
         <ray>
           <scan>
             <horizontal>
-              <samples>1000</samples>
+              <samples>100</samples>
               <resolution>1</resolution>
               <min_angle>-${(M_PI/180)*(81.7/2)}</min_angle>
@@ -43,5 +42,5 @@
             </horizontal>
             <vertical>
-              <samples>10</samples>
+              <samples>100</samples>
               <resolution>1</resolution>
               <min_angle>-${(M_PI/180)*(25.1/2)}</min_angle>
@@ -51,19 +50,16 @@
           <range>
             <min>1</min>
-            <max>260</max>
+            <max>50</max>
             <resolution>0.01</resolution>
           </range>
           <noise>
-            <type>gaussian</type>
-            <mean>0.0</mean>
-            <stddev>0.0</stddev>
-          </noise>
+  	  	    <type>gaussian</type>
+  	  	    <mean>0.0</mean>
+  	  	    <stddev>0.008</stddev>
+  	  	  </noise>
         </ray>
-        <plugin name="gazebo_ros_laser_controller" filename="libgazebo_ros_velodyne_laser.so">
-          <topicName>${name}/points</topicName>
-          <frameName>${name}</frameName>
-          <min_range>1</min_range>
-          <max_range>260</max_range>
-          <gaussianNoise>0.008</gaussianNoise>
+        <plugin name="qev2_lidar_plugin" filename="libhorizon_lidar_plugin.so">
+          <topicName>${name}/pointcloud</topicName>
+          <frameName>${name}_base_link</frameName>
         </plugin>
       </sensor>

File: qutms_autonomous/urdf/sensors/qev2_zed_camera.urdf.xacro (robot description, xacro)
@@ -1,36 +1,36 @@
 <?xml version="1.0"?>
 <robot xmlns:xacro="http://ros.org/wiki/xacro">
-  <xacro:macro name="qev2_zed_camera" params="	*origin
+  	<xacro:macro name="qev2_zed_camera" params="	*origin
                                       	parent:=base_link
                                       	name:=zed_camera">
 		<!-- Camera Base Mount Joint -->
 		<joint name="${name}_base_mount_joint" type="fixed">
-  	  <xacro:insert_block name="origin" />
-  	  <parent link="${parent}"/>
-  	  <child link="${name}_base_link"/>
-  	</joint>
+  	  		<xacro:insert_block name="origin" />
+  	  		<parent link="${parent}"/>
+  	  		<child link="${name}_base_link"/>
+  		</joint>
 		<!-- Camera Base -->
-  	<link name="${name}_base_link">
-			<inertial>
-  	    <mass value="0.135" />
-				<origin xyz="0 0 0"/>
-  	    <inertia ixx="0.00000110261" ixy="0" ixz="0" iyy="0.00003751945" iyz="0" izz="0.00003100781" />
-  	  </inertial>
-  	  <visual>
-  	    <origin xyz="0 0 0" rpy="0 0 0" />
-  	    <geometry>
-  	      <box size="0.03 0.175 0.033" />
-  	    </geometry>
-  	  </visual>
-  	  <collision>
-  	    <origin xyz="0 0 0" rpy="0 0 0"  />
-  	    <geometry>
-  	      <box size="0.03 2.0 0.033" />
-  	    </geometry>
-  	  </collision>
-  	</link>
+  		<link name="${name}_base_link">
+		<inertial>
+  	    	<mass value="0.135" />
+			<origin xyz="0 0 0"/>
+  	    	<inertia ixx="0.00000110261" ixy="0" ixz="0" iyy="0.00003751945" iyz="0" izz="0.00003100781" />
+  	  	</inertial>
+  	  	<visual>
+  	    	<origin xyz="0 0 0" rpy="0 0 0" />
+  	    	<geometry>
+  	    	  <box size="0.03 0.175 0.033" />
+  	    	</geometry>
+  	  	</visual>
+  	  	<collision>
+  	    	<origin xyz="0 0 0" rpy="0 0 0"  />
+  	    	<geometry>
+  	      	<box size="0.03 2.0 0.033" />
+  	    	</geometry>
+  	  	</collision>
+  		</link>
 		<gazebo reference="${name}_base_link">
 			<sensor type="multicamera" name="${name}">
-  	  	<update_rate>30.0</update_rate>
+  	  			<update_rate>30.0</update_rate>
 				<camera name="z-left">
 					<pose>0 0.06 0 0 0 0</pose>
@@ -46,8 +46,8 @@
 					</clip>
 					<noise>
-  	  	      <type>gaussian</type>
-  	  	      <mean>0.0</mean>
-  	  	      <stddev>0.007</stddev>
-  	  	  </noise>
+  	  	      			<type>gaussian</type>
+  	  	      			<mean>0.0</mean>
+  	  	      			<stddev>0.007</stddev>
+  	  	  			</noise>
 				</camera>
 				<camera name="z-right">
@@ -64,25 +64,25 @@
 					</clip>
 					<noise>
-  	  	      <type>gaussian</type>
-  	  	      <mean>0.0</mean>
-  	  	      <stddev>0.007</stddev>
-  	  	  </noise>
+  	  	      			<type>gaussian</type>
+  	  	      			<mean>0.0</mean>
+  	  	      			<stddev>0.007</stddev>
+  	  	  			</noise>
 				</camera>
-  			<plugin name="qev2_camera_plugin" filename="libgazebo_ros_multicamera.so">
+  				<plugin name="qev2_camera_plugin" filename="libgazebo_ros_multicamera.so">
 					<alwaysOn>true</alwaysOn>
 					<updateRate>0.0</updateRate>
 					<cameraName>${name}</cameraName>
-  	  	  <imageTopicName>image_raw</imageTopicName>
-  	  	  <cameraInfoTopicName>camera_info</cameraInfoTopicName>
-  	  	  <frameName>${name}_base_link</frameName>
-  	  	  <hackBaseline>0.07</hackBaseline>
-  	  	  <distortionK1>0.0</distortionK1>
-  	  	  <distortionK2>0.0</distortionK2>
-  	  	  <distortionK3>0.0</distortionK3>
-  	  	  <distortionT1>0.0</distortionT1>
-  	  	  <distortionT2>0.0</distortionT2>
-  			</plugin>
+  	  	  			<imageTopicName>image_raw</imageTopicName>
+  	  	  			<cameraInfoTopicName>camera_info</cameraInfoTopicName>
+  	  	  			<frameName>${name}_base_link</frameName>
+  	  	  			<hackBaseline>0.07</hackBaseline>
+  	  	  			<distortionK1>0.0</distortionK1>
+  	  	  			<distortionK2>0.0</distortionK2>
+  	  	  			<distortionK3>0.0</distortionK3>
+  	  	  			<distortionT1>0.0</distortionT1>
+  	  	  			<distortionT2>0.0</distortionT2>
+  				</plugin>
 			</sensor>
-  	</gazebo>
-  </xacro:macro>
+  		</gazebo>
+  	</xacro:macro>
 </robot>
