Commit message: colour sensors orange to make it fun

File: qutms_description/sensors/gps.urdf.xacro (robot description, xacro)
@@ -28,4 +28,7 @@
 			</collision>
 		</link>
+		<gazebo reference="${name}_base_footprint">
+			<material>Gazebo/Orange</material>
+		</gazebo>
 		<gazebo>
 			<plugin name="gps_plugin" filename="libhector_gazebo_ros_gps.so">

File: qutms_description/sensors/horizon_lidar.urdf.xacro (robot description, xacro)
@@ -6,7 +6,7 @@
             <xacro:insert_block name="origin" />
             <parent link="${parent}"/>
-            <child link="${name}base_footprint"/>
+            <child link="${name}_base_footprint"/>
         </joint>
-        <link name="${name}base_footprint">
+        <link name="${name}_base_footprint">
             <inertial>
                 <mass value="1.18"/>
@@ -26,5 +26,6 @@
             </collision>
         </link>
-        <gazebo reference="${name}base_footprint">
+        <gazebo reference="${name}_base_footprint">
+            <material>Gazebo/Orange</material>
             <sensor type="ray" name="${name}_sensor">
                 <pose>0 0 0 0 0 0</pose>
@@ -57,5 +58,5 @@
                     </noise>
                 </ray>
-                <plugin name="lidar_plugin" filename="libhorizon_lidar_plugin.so">
+                <plugin name="horizon_lidar_plugin" filename="libhorizon_lidar_plugin.so">
                     <robotNamespace>qev</robotNamespace>
                     <topicName>${name}/pointcloud</topicName>

File: qutms_description/sensors/imu.urdf.xacro (robot description, xacro)
@@ -29,4 +29,5 @@
 		</link>
 		<gazebo>
+			<material>Gazebo/Orange</material>
 			<plugin name="imu_plugin" filename="libhector_gazebo_ros_imu.so">
 				<robotNamespace>qev</robotNamespace>

File: qutms_description/sensors/zed_camera.urdf.xacro (robot description, xacro)
@@ -29,4 +29,5 @@
 		</link>
 		<gazebo reference="${name}_base_footprint">
+			<material>Gazebo/Orange</material>
 			<sensor type="multicamera" name="${name}">
 				<update_rate>30.0</update_rate>
