Commit message: Added sensors to model

File: qutms_description/qev/qev.urdf.xacro (robot description, xacro)
@@ -1,4 +1,5 @@
 <?xml version="1.0"?>
-<robot name="qev" xmlns:xacro="http://www.ros.org/wiki/xacro">
+<robot xmlns:xacro="http://www.ros.org/wiki/xacro" name="qev">
+  <xacro:property name="M_PI" value="3.1415926535897931" />
     <!-- ***************** -->
     <!-- Config parameters -->
@@ -15,4 +16,12 @@
     <!--  Include the plugins  -->
     <xacro:include filename="$(find qutms_description)/urdf/plugins.gazebo.xacro"/>
+    <!-- GPS -->
+    <xacro:include filename="$(find qutms_description)/urdf/sensors/qev2_gps.urdf.xacro" />
+    <!-- IMU -->
+    <xacro:include filename="$(find qutms_description)/urdf/sensors/qev2_imu.urdf.xacro" />
+    <!-- LIDAR -->
+    <xacro:include filename="$(find qutms_description)/urdf/sensors/qev2_horizon_lidar.urdf.xacro"/>
+    <!-- Camera -->
+    <xacro:include filename="$(find qutms_description)/urdf/sensors/qev2_zed_camera.urdf.xacro" />
     <!-- ************** -->
     <!-- Robot Elements -->
@@ -24,3 +33,19 @@
     <!-- Wheels -->
     <xacro:wheels chassis_width="2" wheelbase="2.0"/>
+    <!-- GPS -->
+    <xacro:qev2_gps parent="base_footprint" >
+      <origin xyz="0 0 0.71" rpy="0 0 0" />
+    </xacro:qev2_gps>
+    <!-- IMU -->
+    <xacro:qev2_imu parent="base_footprint" >
+      <origin xyz="0 0 0" rpy="0 0 ${M_PI/2}" />
+    </xacro:qev2_imu>
+    <!-- LiDAR -->
+    <xacro:qev2_horizon_lidar parent="base_footprint">
+      <origin xyz="1.1 0 0.1" rpy="0 0 0" />
+    </xacro:qev2_horizon_lidar>
+    <!-- Camera -->
+    <xacro:qev2_zed_camera parent="base_footprint">
+      <origin xyz="-0.4 0 1.3" rpy="0 0 0" />
+    </xacro:qev2_zed_camera>
 </robot>

File: qutms_description/urdf/sensors/qev2_horizon_lidar.urdf.xacro (robot description, xacro)
@@ -8,7 +8,7 @@
       <xacro:insert_block name="origin" />
       <parent link="${parent}"/>
-      <child link="${name}_base_link"/>
+      <child link="${name}base_footprint"/>
     </joint>
-    <link name="${name}_base_link">
+    <link name="${name}base_footprint">
       <inertial>
         <mass value="1.18"/>
@@ -28,5 +28,5 @@
       </collision>
     </link>
-    <gazebo reference="${name}_base_link">
+    <gazebo reference="${name}base_footprint">
       <sensor type="ray" name="${name}_sensor">
         <pose>0 0 0 0 0 0</pose>
@@ -61,5 +61,5 @@
         <plugin name="qev2_lidar_plugin" filename="libhorizon_lidar_plugin.so">
           <topicName>${name}/pointcloud</topicName>
-          <frameName>${name}_base_link</frameName>
+          <frameName>${name}_base_footprint</frameName>
         </plugin>
       </sensor>

File: qutms_description/urdf/sensors/qev2_imu.urdf.xacro (robot description, xacro)
@@ -10,8 +10,8 @@
       <xacro:insert_block name="origin" />
       <parent link="${parent}"/>
-      <child link="${name}_base_link"/>
+      <child link="${name}_base_footprint"/>
   	</joint>
 		<!-- IMU Base -->
-    <link name="${name}_base_link">
+    <link name="${name}_base_footprint">
 			<inertial>
         <mass value="0.385" />
@@ -34,7 +34,7 @@
 	<gazebo>
   	  <plugin name="imu_controller_${name}" filename="libhector_gazebo_ros_imu.so">
-  	    <robotNamespace>$(arg robot_namespace)</robotNamespace>
+  	    <robotNamespace>qev</robotNamespace>
   	    <updateRate>${update_rate}</updateRate>
-  	    <bodyName>${name}_base_link</bodyName>
+  	    <bodyName>${name}_base_footprint</bodyName>
   	    <topicName>${topic_name}</topicName>
   	    <accelDrift>0.005 0.005 0.005</accelDrift>

File: qutms_description/urdf/sensors/qev2_zed_camera.urdf.xacro (robot description, xacro)
@@ -8,8 +8,8 @@
   	  		<xacro:insert_block name="origin" />
   	  		<parent link="${parent}"/>
-  	  		<child link="${name}_base_link"/>
+  	  		<child link="${name}_base_footprint"/>
   		</joint>
 		<!-- Camera Base -->
-  		<link name="${name}_base_link">
+  		<link name="${name}_base_footprint">
 		<inertial>
   	    	<mass value="0.135" />
@@ -75,5 +75,5 @@
   	  	  			<imageTopicName>image_raw</imageTopicName>
   	  	  			<cameraInfoTopicName>camera_info</cameraInfoTopicName>
-  	  	  			<frameName>${name}_base_link</frameName>
+  	  	  			<frameName>${name}_base_footprint</frameName>
   	  	  			<hackBaseline>0.07</hackBaseline>
   	  	  			<distortionK1>0.0</distortionK1>
