Commit message: format all xmls consistently

File: qutms_description/qev/qev.urdf.xacro (robot description, xacro)
@@ -1,5 +1,5 @@
 <?xml version="1.0"?>
 <robot xmlns:xacro="http://www.ros.org/wiki/xacro" name="qev">
-  <xacro:property name="M_PI" value="3.1415926535897931" />
+    <xacro:property name="M_PI" value="3.1415926535897931" />
     <!-- ***************** -->
     <!-- Config parameters -->
@@ -28,24 +28,22 @@
     <!-- ************** -->
     <!-- Chassis of the car -->
-    <xacro:car_base chassis_length="2.165"
-                    chassis_width="0.735"
-                    chassis_height="0.63"/>
+    <xacro:car_base chassis_length="2.165" chassis_width="0.735" chassis_height="0.63"/>
     <!-- Wheels -->
     <xacro:wheels chassis_width="2" wheelbase="2.0"/>
     <!-- GPS -->
-    <xacro:qev2_gps parent="base_footprint" >
-      <origin xyz="0 0 0.71" rpy="0 0 0" />
+    <xacro:qev2_gps parent="base_footprint">
+        <origin xyz="0 0 0.71" rpy="0 0 0" />
     </xacro:qev2_gps>
     <!-- IMU -->
-    <xacro:qev2_imu parent="base_footprint" >
-      <origin xyz="0 0 0" rpy="0 0 ${M_PI/2}" />
+    <xacro:qev2_imu parent="base_footprint">
+        <origin xyz="0 0 0" rpy="0 0 ${M_PI/2}" />
     </xacro:qev2_imu>
     <!-- LiDAR -->
     <xacro:qev2_horizon_lidar parent="base_footprint">
-      <origin xyz="1.1 0 0.1" rpy="0 0 0" />
+        <origin xyz="1.1 0 0.1" rpy="0 0 0" />
     </xacro:qev2_horizon_lidar>
     <!-- Camera -->
     <xacro:qev2_zed_camera parent="base_footprint">
-      <origin xyz="-0.4 0 1.3" rpy="0 0 0" />
+        <origin xyz="-0.4 0 1.3" rpy="0 0 0" />
     </xacro:qev2_zed_camera>
 </robot>

File: qutms_description/urdf/car_base.urdf.xacro (robot description, xacro)
@@ -1,40 +1,33 @@
 <?xml version="1.0"?>
-<robot name="base" xmlns:xacro="http://www.ros.org/wiki/xacro">
-  <xacro:macro name="car_base"
-               params="chassis_width chassis_length chassis_height">
-    <!-- BASE FOOTPRINT -->
-    <link name="base_footprint"/>
-    <joint name="chassis_joint" type="fixed">
-      <parent link="base_footprint"/>
-      <child link="chassis"/>
-      <origin xyz="0 0 0"
-              rpy="0 0 0"/>
-      <axis xyz="1 0 0"/>
-    </joint>
-    <link name="chassis">
-      <visual>
-        <origin xyz="0 0 0" rpy="0 0 0" />
-        <geometry>
-          <box size="${chassis_length} ${chassis_width} ${chassis_height}"/>
-        </geometry>
-      </visual>
-      <inertial>
-        <origin xyz="0 0 0" rpy="0 0 0" />
-        <mass value="140" />
-        <inertia
-            ixx="16.3"
-            ixy="0"
-            ixz="0"
-            iyy="33.6"
-            iyz="0"
-            izz="47.9" />
-      </inertial>
-      <collision>
-        <origin xyz="0 0 0" rpy="0 0 0" />
-        <geometry>
-          <box size="${chassis_length} ${chassis_width} ${chassis_height}"/>
-        </geometry>
-      </collision>
-    </link>
-  </xacro:macro>
+<robot name="base"
+    xmlns:xacro="http://www.ros.org/wiki/xacro">
+    <xacro:macro name="car_base" params="chassis_width chassis_length chassis_height">
+        <!-- BASE FOOTPRINT -->
+        <link name="base_footprint"/>
+        <joint name="chassis_joint" type="fixed">
+            <parent link="base_footprint"/>
+            <child link="chassis"/>
+            <origin xyz="0 0 0" rpy="0 0 0"/>
+            <axis xyz="1 0 0"/>
+        </joint>
+        <link name="chassis">
+            <visual>
+                <origin xyz="0 0 0" rpy="0 0 0" />
+                <geometry>
+                    <box size="${chassis_length} ${chassis_width} ${chassis_height}"/>
+                </geometry>
+            </visual>
+            <inertial>
+                <origin xyz="0 0 0" rpy="0 0 0" />
+                <mass value="140" />
+                <inertia ixx="16.3" ixy="0" ixz="0" iyy="33.6" iyz="0" izz="47.9" />
+            </inertial>
+            <collision>
+                <origin xyz="0 0 0" rpy="0 0 0" />
+                <geometry>
+                    <box size="${chassis_length} ${chassis_width} ${chassis_height}"/>
+                </geometry>
+            </collision>
+        </link>
+    </xacro:macro>
 </robot>

File: qutms_description/urdf/plugins.gazebo.xacro (robot description, xacro)
@@ -1,32 +1,32 @@
 <?xml version="1.0"?>
 <robot xmlns:xacro="http://www.ros.org/wiki/xacro">
-  <xacro:arg name="publish_tf" default="false"/>
-  <!-- Custom plugin which controls the car using a given vehicle model.
+    <xacro:arg name="publish_tf" default="false"/>
+    <!-- Custom plugin which controls the car using a given vehicle model.
    It controls the car by setting its velocity and position
    and the steering angle of the wheels -->
-  <gazebo>
-    <plugin name="race_car" filename="libgazebo_race_car_model.so">
-      <update_rate>1000.0</update_rate>
-      <publish_rate>200.0</publish_rate>
-      <vehicle_model>$(arg vehicle_model)</vehicle_model>
-      <front_left_wheel_steering>left_steering_hinge_joint</front_left_wheel_steering>
-      <front_right_wheel_steering>right_steering_hinge_joint</front_right_wheel_steering>
-      <front_left_wheel>front_left_wheel_joint</front_left_wheel>
-      <front_right_wheel>front_right_wheel_joint</front_right_wheel>
-      <rear_left_wheel>rear_left_wheel_joint</rear_left_wheel>
-      <rear_right_wheel>rear_right_wheel_joint</rear_right_wheel>
-      <yaml_config>$(arg config_file)</yaml_config>
-      <referenceFrame>map</referenceFrame>
-      <robotFrame>base_footprint</robotFrame>
-      <publishTransform>$(arg publish_tf)</publishTransform>
-      <stateTopicName>/ground_truth/state</stateTopicName>
-      <wheelSpeedsTopicName>/ros_can/wheel_speeds</wheelSpeedsTopicName>
-      <odometryTopicName>/ground_truth/odom</odometryTopicName>
-      <positionNoise>0.0 0.0 0.0</positionNoise>
-      <orientationNoise>0.0 0.0 0.0</orientationNoise> <!-- Yaw Pitch Roll -->
-      <linearVelocityNoise>0.0 0.0 0.0</linearVelocityNoise>
-      <angularVelocityNoise>0.0 0.0 0.0</angularVelocityNoise>  <!-- X Y Z -->
-      <linearAccelerationNoise>0.0 0.0 0.0</linearAccelerationNoise>
-    </plugin>
-  </gazebo>
+    <gazebo>
+        <plugin name="race_car" filename="libgazebo_race_car_model.so">
+            <update_rate>1000.0</update_rate>
+            <publish_rate>200.0</publish_rate>
+            <vehicle_model>$(arg vehicle_model)</vehicle_model>
+            <front_left_wheel_steering>left_steering_hinge_joint</front_left_wheel_steering>
+            <front_right_wheel_steering>right_steering_hinge_joint</front_right_wheel_steering>
+            <front_left_wheel>front_left_wheel_joint</front_left_wheel>
+            <front_right_wheel>front_right_wheel_joint</front_right_wheel>
+            <rear_left_wheel>rear_left_wheel_joint</rear_left_wheel>
+            <rear_right_wheel>rear_right_wheel_joint</rear_right_wheel>
+            <yaml_config>$(arg config_file)</yaml_config>
+            <referenceFrame>map</referenceFrame>
+            <robotFrame>base_footprint</robotFrame>
+            <publishTransform>$(arg publish_tf)</publishTransform>
+            <stateTopicName>/ground_truth/state</stateTopicName>
+            <wheelSpeedsTopicName>/ros_can/wheel_speeds</wheelSpeedsTopicName>
+            <odometryTopicName>/ground_truth/odom</odometryTopicName>
+            <positionNoise>0.0 0.0 0.0</positionNoise>
+            <orientationNoise>0.0 0.0 0.0</orientationNoise>            <!-- Yaw Pitch Roll -->
+            <linearVelocityNoise>0.0 0.0 0.0</linearVelocityNoise>
+            <angularVelocityNoise>0.0 0.0 0.0</angularVelocityNoise>            <!-- X Y Z -->
+            <linearAccelerationNoise>0.0 0.0 0.0</linearAccelerationNoise>
+        </plugin>
+    </gazebo>
 </robot>

File: qutms_description/urdf/sensors/qev2_gps.urdf.xacro (robot description, xacro)
@@ -1,50 +1,46 @@
 <?xml version="1.0"?>
 <robot xmlns:xacro="http://ros.org/wiki/xacro">
-  <xacro:macro name="qev2_gps" params="	*origin
-                                      	parent:=base_footprint
-                                      	name:=gps
-                                      	topic_name:=gps/data
-                                      	update_rate:=30.0">
-	<!-- GPS Base Mount Joint -->
-	<joint name="${name}_base_mount_joint" type="fixed">
-    <xacro:insert_block name="origin" />
-    <parent link="${parent}"/>
-    <child link="${name}_base_footprint"/>
-  </joint>
-	<!-- GPS Base -->
-  <link name="${name}_base_footprint">
-		<inertial>
-      <mass value="0.8" />
-			<origin xyz="0 0 0"/>
-      <inertia ixx="0.016" ixy="0" ixz="0" iyy="0.049" iyz="0" izz="0.049" />
-    </inertial>
-    <visual>
-      <origin xyz="0 0 0" rpy="0 0 0" />
-      <geometry>
-        <cylinder length="0.05" radius="0.2" />
-      </geometry>
-    </visual>
-    <collision>
-      <origin xyz="0 0 0" rpy="0 0 0"  />
-      <geometry>
-        <cylinder length="0.05" radius="0.2" />
-      </geometry>
-    </collision>
-  </link>
-	<gazebo>
-  	  <plugin name="gps_controller_${name}" filename="libhector_gazebo_ros_gps.so">
-  	    <robotNamespace>qev</robotNamespace>
-  	    <updateRate>30</updateRate>
-  	    <bodyName>${name}_base_footprint</bodyName>
-  	    <frameId>${name}_base_footprint</frameId>
-  	    <topicName>${topic_name}</topicName>
-  	    <velocityTopicName>gps/vel</velocityTopicName>
-  	    <referenceLatitude>49.9</referenceLatitude>
-  	    <referenceLongitude>8.9</referenceLongitude>
-  	    <referenceHeading>0</referenceHeading>
-  	    <referenceAltitude>0</referenceAltitude>
-  	    <drift>0.0001 0.0001 0.0001</drift>
-  	  </plugin>
-  	</gazebo>
-  </xacro:macro>
+	<xacro:macro name="qev2_gps" params="*origin parent:=base_footprint name:=gps topic_name:=gps/data update_rate:=30.0">
+		<!-- GPS Base Mount Joint -->
+		<joint name="${name}_base_mount_joint" type="fixed">
+			<xacro:insert_block name="origin"/>
+			<parent link="${parent}"/>
+			<child link="${name}_base_footprint"/>
+		</joint>
+		<!-- GPS Base -->
+		<link name="${name}_base_footprint">
+			<inertial>
+				<mass value="0.8" />
+				<origin xyz="0 0 0"/>
+				<inertia ixx="0.016" ixy="0" ixz="0" iyy="0.049" iyz="0" izz="0.049" />
+			</inertial>
+			<visual>
+				<origin xyz="0 0 0" rpy="0 0 0" />
+				<geometry>
+					<cylinder length="0.05" radius="0.2" />
+				</geometry>
+			</visual>
+			<collision>
+				<origin xyz="0 0 0" rpy="0 0 0" />
+				<geometry>
+					<cylinder length="0.05" radius="0.2" />
+				</geometry>
+			</collision>
+		</link>
+		<gazebo>
+			<plugin name="gps_controller_${name}" filename="libhector_gazebo_ros_gps.so">
+				<robotNamespace>qev</robotNamespace>
+				<updateRate>30</updateRate>
+				<bodyName>${name}_base_footprint</bodyName>
+				<frameId>${name}_base_footprint</frameId>
+				<topicName>${topic_name}</topicName>
+				<velocityTopicName>gps/vel</velocityTopicName>
+				<referenceLatitude>49.9</referenceLatitude>
+				<referenceLongitude>8.9</referenceLongitude>
+				<referenceHeading>0</referenceHeading>
+				<referenceAltitude>0</referenceAltitude>
+				<drift>0.0001 0.0001 0.0001</drift>
+			</plugin>
+		</gazebo>
+	</xacro:macro>
 </robot>

File: qutms_description/urdf/sensors/qev2_horizon_lidar.urdf.xacro (robot description, xacro)
@@ -1,68 +1,66 @@
 <?xml version="1.0"?>
 <robot xmlns:xacro="http://ros.org/wiki/xacro" name="Horizon">
-  <xacro:property name="M_PI" value="3.1415926535897931" />
-  <xacro:macro name="qev2_horizon_lidar" params=" *origin
-                                      parent:=base_footprint
-                                      name:=horizon_lidar">
-    <joint name="${name}_base_mount_joint" type="fixed">
-      <xacro:insert_block name="origin" />
-      <parent link="${parent}"/>
-      <child link="${name}base_footprint"/>
-    </joint>
-    <link name="${name}base_footprint">
-      <inertial>
-        <mass value="1.18"/>
-        <origin xyz="0 0 0" rpy="0 0 0" />
-        <inertia ixx="0.00199429833" ixy="0" ixz="0" iyy="0.00188347666" iyz="0" izz="0.00127685833"/>
-      </inertial>
-      <visual>
-        <geometry>
-          <box size="0.115 0.077 0.084"/>
-        </geometry>
-      </visual>
-      <collision>
-        <origin xyz="0 0 0" rpy="0 0 0" />
-        <geometry>
-          <box size="0.115 0.077 0.084"/>
-        </geometry>
-      </collision>
-    </link>
-    <gazebo reference="${name}base_footprint">
-      <sensor type="ray" name="${name}_sensor">
-        <pose>0 0 0 0 0 0</pose>
-        <update_rate>30.0</update_rate>
-        <visualize>false</visualize>
-        <ray>
-          <scan>
-            <horizontal>
-              <samples>100</samples>
-              <resolution>1</resolution>
-              <min_angle>-${(M_PI/180)*(81.7/2)}</min_angle>
-              <max_angle>${(M_PI/180)*(81.7/2)}</max_angle>
-            </horizontal>
-            <vertical>
-              <samples>100</samples>
-              <resolution>1</resolution>
-              <min_angle>-${(M_PI/180)*(25.1/2)}</min_angle>
-              <max_angle>${(M_PI/180)*(25.1/2)}</max_angle>
-            </vertical>
-          </scan>
-          <range>
-            <min>1</min>
-            <max>50</max>
-            <resolution>0.01</resolution>
-          </range>
-          <noise>
-  	  	    <type>gaussian</type>
-  	  	    <mean>0.0</mean>
-  	  	    <stddev>0.008</stddev>
-  	  	  </noise>
-        </ray>
-        <plugin name="qev2_lidar_plugin" filename="libhorizon_lidar_plugin.so">
-          <topicName>${name}/pointcloud</topicName>
-          <frameName>${name}_base_footprint</frameName>
-        </plugin>
-      </sensor>
-    </gazebo>
-  </xacro:macro>
+    <xacro:property name="M_PI" value="3.1415926535897931" />
+    <xacro:macro name="qev2_horizon_lidar" params=" *origin parent:=base_footprint name:=horizon_lidar">
+        <joint name="${name}_base_mount_joint" type="fixed">
+            <xacro:insert_block name="origin" />
+            <parent link="${parent}"/>
+            <child link="${name}base_footprint"/>
+        </joint>
+        <link name="${name}base_footprint">
+            <inertial>
+                <mass value="1.18"/>
+                <origin xyz="0 0 0" rpy="0 0 0" />
+                <inertia ixx="0.00199429833" ixy="0" ixz="0" iyy="0.00188347666" iyz="0" izz="0.00127685833"/>
+            </inertial>
+            <visual>
+                <geometry>
+                    <box size="0.115 0.077 0.084"/>
+                </geometry>
+            </visual>
+            <collision>
+                <origin xyz="0 0 0" rpy="0 0 0" />
+                <geometry>
+                    <box size="0.115 0.077 0.084"/>
+                </geometry>
+            </collision>
+        </link>
+        <gazebo reference="${name}base_footprint">
+            <sensor type="ray" name="${name}_sensor">
+                <pose>0 0 0 0 0 0</pose>
+                <update_rate>30.0</update_rate>
+                <visualize>false</visualize>
+                <ray>
+                    <scan>
+                        <horizontal>
+                            <samples>100</samples>
+                            <resolution>1</resolution>
+                            <min_angle>-${(M_PI/180)*(81.7/2)}</min_angle>
+                            <max_angle>${(M_PI/180)*(81.7/2)}</max_angle>
+                        </horizontal>
+                        <vertical>
+                            <samples>100</samples>
+                            <resolution>1</resolution>
+                            <min_angle>-${(M_PI/180)*(25.1/2)}</min_angle>
+                            <max_angle>${(M_PI/180)*(25.1/2)}</max_angle>
+                        </vertical>
+                    </scan>
+                    <range>
+                        <min>1</min>
+                        <max>50</max>
+                        <resolution>0.01</resolution>
+                    </range>
+                    <noise>
+                        <type>gaussian</type>
+                        <mean>0.0</mean>
+                        <stddev>0.008</stddev>
+                    </noise>
+                </ray>
+                <plugin name="qev2_lidar_plugin" filename="libhorizon_lidar_plugin.so">
+                    <topicName>${name}/pointcloud</topicName>
+                    <frameName>${name}_base_footprint</frameName>
+                </plugin>
+            </sensor>
+        </gazebo>
+    </xacro:macro>
 </robot>

File: qutms_description/urdf/sensors/qev2_imu.urdf.xacro (robot description, xacro)
@@ -1,49 +1,45 @@
 <?xml version="1.0"?>
 <robot xmlns:xacro="http://ros.org/wiki/xacro">
-	<xacro:macro name="qev2_imu" params="	*origin
-                                      	parent:=base_footprint
-                                      	name:=imu
-                                      	topic_name:=imu/data
-                                      	update_rate:=30.0">
+	<xacro:macro name="qev2_imu" params="*origin parent:=base_footprint name:=imu topic_name:=imu/data update_rate:=30.0">
 		<!-- IMU Base Mount Joint -->
 		<joint name="${name}_base_mount_joint" type="fixed">
-      <xacro:insert_block name="origin" />
-      <parent link="${parent}"/>
-      <child link="${name}_base_footprint"/>
-  	</joint>
+			<xacro:insert_block name="origin" />
+			<parent link="${parent}"/>
+			<child link="${name}_base_footprint"/>
+		</joint>
 		<!-- IMU Base -->
-    <link name="${name}_base_footprint">
+		<link name="${name}_base_footprint">
 			<inertial>
-        <mass value="0.385" />
+				<mass value="0.385" />
 				<origin xyz="0 0 0"/>
-        <inertia ixx="0.00000008608" ixy="0" ixz="0" iyy="0.00000033679" iyz="0" izz="0.00000860809" />
-      </inertial>
-      <visual>
-        <origin xyz="0 0 0" rpy="0 0 0" />
-        <geometry>
-          <box size="0.18 0.091 0.018"/>
-        </geometry>
-      </visual>
-      <collision>
-        <origin xyz="0 0 0" rpy="0 0 0"  />
-        <geometry>
-          <box size="0.18 0.091 0.018"/>
-        </geometry>
-      </collision>
-    </link>
-	<gazebo>
-  	  <plugin name="imu_controller_${name}" filename="libhector_gazebo_ros_imu.so">
-  	    <robotNamespace>qev</robotNamespace>
-  	    <updateRate>${update_rate}</updateRate>
-  	    <bodyName>${name}_base_footprint</bodyName>
-  	    <topicName>${topic_name}</topicName>
-  	    <accelDrift>0.005 0.005 0.005</accelDrift>
-  	    <accelGaussianNoise>0.005 0.005 0.005</accelGaussianNoise>
-  	    <rateDrift>0.005 0.005 0.005 </rateDrift>
-  	    <rateGaussianNoise>0.005 0.005 0.005 </rateGaussianNoise>
-  	    <headingDrift>0.005</headingDrift>
-  	    <headingGaussianNoise>0.005</headingGaussianNoise>
-  	  </plugin>
-  	</gazebo>
+				<inertia ixx="0.00000008608" ixy="0" ixz="0" iyy="0.00000033679" iyz="0" izz="0.00000860809" />
+			</inertial>
+			<visual>
+				<origin xyz="0 0 0" rpy="0 0 0" />
+				<geometry>
+					<box size="0.18 0.091 0.018"/>
+				</geometry>
+			</visual>
+			<collision>
+				<origin xyz="0 0 0" rpy="0 0 0" />
+				<geometry>
+					<box size="0.18 0.091 0.018"/>
+				</geometry>
+			</collision>
+		</link>
+		<gazebo>
+			<plugin name="imu_controller_${name}" filename="libhector_gazebo_ros_imu.so">
+				<robotNamespace>qev</robotNamespace>
+				<updateRate>${update_rate}</updateRate>
+				<bodyName>${name}_base_footprint</bodyName>
+				<topicName>${topic_name}</topicName>
+				<accelDrift>0.005 0.005 0.005</accelDrift>
+				<accelGaussianNoise>0.005 0.005 0.005</accelGaussianNoise>
+				<rateDrift>0.005 0.005 0.005 </rateDrift>
+				<rateGaussianNoise>0.005 0.005 0.005 </rateGaussianNoise>
+				<headingDrift>0.005</headingDrift>
+				<headingGaussianNoise>0.005</headingGaussianNoise>
+			</plugin>
+		</gazebo>
 	</xacro:macro>
 </robot>
