Commit message: format all xmls consistently

File: qutms_description/urdf/sensors/qev2_zed_camera.urdf.xacro (robot description, xacro)
@@ -1,53 +1,51 @@
 <?xml version="1.0"?>
 <robot xmlns:xacro="http://ros.org/wiki/xacro">
-  	<xacro:macro name="qev2_zed_camera" params="	*origin
-                                      	parent:=base_footprint
-                                      	name:=zed_camera">
+	<xacro:macro name="qev2_zed_camera" params="*origin parent:=base_footprint name:=zed_camera">
 		<!-- Camera Base Mount Joint -->
 		<joint name="${name}_base_mount_joint" type="fixed">
-  	  		<xacro:insert_block name="origin" />
-  	  		<parent link="${parent}"/>
-  	  		<child link="${name}_base_footprint"/>
-  		</joint>
+			<xacro:insert_block name="origin" />
+			<parent link="${parent}"/>
+			<child link="${name}_base_footprint"/>
+		</joint>
 		<!-- Camera Base -->
-  		<link name="${name}_base_footprint">
-		<inertial>
-  	    	<mass value="0.135" />
-			<origin xyz="0 0 0"/>
-  	    	<inertia ixx="0.00000110261" ixy="0" ixz="0" iyy="0.00003751945" iyz="0" izz="0.00003100781" />
-  	  	</inertial>
-  	  	<visual>
-  	    	<origin xyz="0 0 0" rpy="0 0 0" />
-  	    	<geometry>
-  	    	  <box size="0.03 0.175 0.033" />
-  	    	</geometry>
-  	  	</visual>
-  	  	<collision>
-  	    	<origin xyz="0 0 0" rpy="0 0 0"  />
-  	    	<geometry>
-  	      	<box size="0.03 2.0 0.033" />
-  	    	</geometry>
-  	  	</collision>
-  		</link>
+		<link name="${name}_base_footprint">
+			<inertial>
+				<mass value="0.135" />
+				<origin xyz="0 0 0"/>
+				<inertia ixx="0.00000110261" ixy="0" ixz="0" iyy="0.00003751945" iyz="0" izz="0.00003100781" />
+			</inertial>
+			<visual>
+				<origin xyz="0 0 0" rpy="0 0 0" />
+				<geometry>
+					<box size="0.03 0.175 0.033" />
+				</geometry>
+			</visual>
+			<collision>
+				<origin xyz="0 0 0" rpy="0 0 0" />
+				<geometry>
+					<box size="0.03 2.0 0.033" />
+				</geometry>
+			</collision>
+		</link>
 		<gazebo reference="${name}_base_link">
 			<sensor type="multicamera" name="${name}">
-  	  			<update_rate>30.0</update_rate>
+				<update_rate>30.0</update_rate>
 				<camera name="z-left">
 					<pose>0 0.06 0 0 0 0</pose>
 					<horizontal_fov>1.5707963268</horizontal_fov>
 					<image>
-		  			<width>3840</width>
-		  			<height>1080</height>
-		  			<format>R8G8B8</format>
+						<width>3840</width>
+						<height>1080</height>
+						<format>R8G8B8</format>
 					</image>
 					<clip>
-		  			<near>0.5</near>
-		  			<far>25</far>
+						<near>0.5</near>
+						<far>25</far>
 					</clip>
 					<noise>
-  	  	      			<type>gaussian</type>
-  	  	      			<mean>0.0</mean>
-  	  	      			<stddev>0.007</stddev>
-  	  	  			</noise>
+						<type>gaussian</type>
+						<mean>0.0</mean>
+						<stddev>0.007</stddev>
+					</noise>
 				</camera>
 				<camera name="z-right">
@@ -55,34 +53,34 @@
 					<horizontal_fov>1.5707963268</horizontal_fov>
 					<image>
-		  			<width>3840</width>
-		  			<height>1080</height>
-		  			<format>R8G8B8</format>
+						<width>3840</width>
+						<height>1080</height>
+						<format>R8G8B8</format>
 					</image>
 					<clip>
-		  			<near>0.5</near>
-		  			<far>25</far>
+						<near>0.5</near>
+						<far>25</far>
 					</clip>
 					<noise>
-  	  	      			<type>gaussian</type>
-  	  	      			<mean>0.0</mean>
-  	  	      			<stddev>0.007</stddev>
-  	  	  			</noise>
+						<type>gaussian</type>
+						<mean>0.0</mean>
+						<stddev>0.007</stddev>
+					</noise>
 				</camera>
-  				<plugin name="qev2_camera_plugin" filename="libgazebo_ros_multicamera.so">
+				<plugin name="qev2_camera_plugin" filename="libgazebo_ros_multicamera.so">
 					<alwaysOn>true</alwaysOn>
 					<updateRate>0.0</updateRate>
 					<cameraName>${name}</cameraName>
-  	  	  			<imageTopicName>image_raw</imageTopicName>
-  	  	  			<cameraInfoTopicName>camera_info</cameraInfoTopicName>
-  	  	  			<frameName>${name}_base_footprint</frameName>
-  	  	  			<hackBaseline>0.07</hackBaseline>
-  	  	  			<distortionK1>0.0</distortionK1>
-  	  	  			<distortionK2>0.0</distortionK2>
-  	  	  			<distortionK3>0.0</distortionK3>
-  	  	  			<distortionT1>0.0</distortionT1>
-  	  	  			<distortionT2>0.0</distortionT2>
-  				</plugin>
+					<imageTopicName>image_raw</imageTopicName>
+					<cameraInfoTopicName>camera_info</cameraInfoTopicName>
+					<frameName>${name}_base_footprint</frameName>
+					<hackBaseline>0.07</hackBaseline>
+					<distortionK1>0.0</distortionK1>
+					<distortionK2>0.0</distortionK2>
+					<distortionK3>0.0</distortionK3>
+					<distortionT1>0.0</distortionT1>
+					<distortionT2>0.0</distortionT2>
+				</plugin>
 			</sensor>
-  		</gazebo>
-  	</xacro:macro>
+		</gazebo>
+	</xacro:macro>
 </robot>

File: qutms_description/urdf/wheels.urdf.xacro (robot description, xacro)
@@ -1,116 +1,98 @@
 <?xml version="1.0"?>
-<robot name="wheels" xmlns:xacro="http://www.ros.org/wiki/xacro">
-  <xacro:macro name="wheels"
-               params="chassis_width wheelbase">
-    <!-- ********** -->
-    <!-- Parameters -->
-    <!-- ********** -->
-    <xacro:property name="degrees_90" value="1.5708"/>
-    <xacro:property name="wheel_mass" value="10.0"/>
-    <xacro:property name="wheel_diameter" value="0.505"/>
-    <xacro:property name="wheel_width" value="0.2"/>
-    <xacro:property name="wheel_friction_mu1" value="2"/>
-    <xacro:property name="wheel_friction_mu2" value="2"/>
-    <xacro:property name="wheel_friction_kp" value="1e8"/>
-    <xacro:property name="steering_hinge_mass" value="1"/>
-    <!-- ***************** -->
-    <!-- Wheel description -->
-    <!-- ***************** -->
-    <xacro:macro name="wheel"
-                 params="lr_prefix fr_prefix">
-      <link name="${lr_prefix}_${fr_prefix}_wheel">
-        <inertial>
-          <origin xyz="0 0 0" rpy="0 0 0" />
-          <mass value="${wheel_mass}"/>
-          <inertia
-              ixx="0.3"
-              ixy="0"
-              ixz="0"
-              iyy="0.2"
-              iyz="0"
-              izz="0.2"   />
-        </inertial>
-        <visual>
-          <origin xyz="0 0 0" rpy="${degrees_90} 0 0"/>
-          <geometry>
-            <cylinder radius="${wheel_diameter / 2}" length="${wheel_width}"/>
-          </geometry>
-        </visual>
-        <collision>
-          <origin xyz="0 0 0" rpy="${degrees_90} 0 0"/>
-          <geometry>
-            <cylinder radius="${wheel_diameter / 2}" length="${wheel_width}"/>
-          </geometry>
-        </collision>
-      </link>
-      <gazebo reference="${lr_prefix}_${fr_prefix}_wheel">
-        <material>Gazebo/Black</material>
-        <mu1>${wheel_friction_mu1}</mu1>
-        <mu2>${wheel_friction_mu2}</mu2>
-        <!-- <minDepth>0.005</minDepth> -->
-        <kp>${wheel_friction_kp}</kp>
-      </gazebo>
-    </xacro:macro>
-    <!-- ********************************* -->
-    <!-- Front and rear wheel descriptions -->
-    <!-- ********************************* -->
-    <!-- Description of how a front wheel is connected to the base_footprint -->
-    <xacro:macro name="front_wheel"
-                 params="lr_prefix lr_reflect">
-      <joint name="${lr_prefix}_steering_hinge_joint" type="revolute">
-        <origin xyz="${wheelbase / 2}
+<robot name="wheels"
+	xmlns:xacro="http://www.ros.org/wiki/xacro">
+	<xacro:macro name="wheels" params="chassis_width wheelbase">
+		<!-- ********** -->
+		<!-- Parameters -->
+		<!-- ********** -->
+		<xacro:property name="degrees_90" value="1.5708"/>
+		<xacro:property name="wheel_mass" value="10.0"/>
+		<xacro:property name="wheel_diameter" value="0.505"/>
+		<xacro:property name="wheel_width" value="0.2"/>
+		<xacro:property name="wheel_friction_mu1" value="2"/>
+		<xacro:property name="wheel_friction_mu2" value="2"/>
+		<xacro:property name="wheel_friction_kp" value="1e8"/>
+		<xacro:property name="steering_hinge_mass" value="1"/>
+		<!-- ***************** -->
+		<!-- Wheel description -->
+		<!-- ***************** -->
+		<xacro:macro name="wheel" params="lr_prefix fr_prefix">
+			<link name="${lr_prefix}_${fr_prefix}_wheel">
+				<inertial>
+					<origin xyz="0 0 0" rpy="0 0 0" />
+					<mass value="${wheel_mass}"/>
+					<inertia ixx="0.3" ixy="0" ixz="0" iyy="0.2" iyz="0" izz="0.2" />
+				</inertial>
+				<visual>
+					<origin xyz="0 0 0" rpy="${degrees_90} 0 0"/>
+					<geometry>
+						<cylinder radius="${wheel_diameter / 2}" length="${wheel_width}"/>
+					</geometry>
+				</visual>
+				<collision>
+					<origin xyz="0 0 0" rpy="${degrees_90} 0 0"/>
+					<geometry>
+						<cylinder radius="${wheel_diameter / 2}" length="${wheel_width}"/>
+					</geometry>
+				</collision>
+			</link>
+			<gazebo reference="${lr_prefix}_${fr_prefix}_wheel">
+				<material>Gazebo/Black</material>
+				<mu1>${wheel_friction_mu1}</mu1>
+				<mu2>${wheel_friction_mu2}</mu2>
+				<!-- <minDepth>0.005</minDepth> -->
+				<kp>${wheel_friction_kp}</kp>
+			</gazebo>
+		</xacro:macro>
+		<!-- ********************************* -->
+		<!-- Front and rear wheel descriptions -->
+		<!-- ********************************* -->
+		<!-- Description of how a front wheel is connected to the base_footprint -->
+		<xacro:macro name="front_wheel" params="lr_prefix lr_reflect">
+			<joint name="${lr_prefix}_steering_hinge_joint" type="revolute">
+				<origin xyz="${wheelbase / 2}
                      ${lr_reflect * ((chassis_width - wheel_width) / 2)}
-                     0"
-                rpy="0 0 0"/>
-        <parent link="base_footprint"/>
-        <child link="${lr_prefix}_steering_hinge"/>
-        <axis xyz="0 0 1"/>
-        <limit lower="${config['input_ranges']['steering']['min']}" upper="${config['input_ranges']['steering']['max']}" effort="10000000" velocity="1000000"/>
-      </joint>
-      <link name="${lr_prefix}_steering_hinge">
-        <inertial>
-          <origin xyz="0 0 0" rpy="0 0 0" />
-          <mass value="${steering_hinge_mass}"/>
-          <inertia
-              ixx="0.04"
-              ixy="0.0"
-              ixz="0.0"
-              iyy="0.04"
-              iyz="0.0"
-              izz="0.04"   />
-        </inertial>
-      </link>
-      <joint name="front_${lr_prefix}_wheel_joint" type="continuous">
-        <origin xyz="0 0 0"
-                rpy="0 0 0"/>
-        <parent link="${lr_prefix}_steering_hinge"/>
-        <child link="${lr_prefix}_front_wheel"/>
-        <axis xyz="0 1 0"/>
-        <limit lower="0" upper="0" effort="10000000" velocity="1000000"/>
-      </joint>
-      <xacro:wheel lr_prefix="${lr_prefix}" fr_prefix="front"/>
-    </xacro:macro>
-    <!-- Description of how a rear wheel is connected to the base_footprint -->
-    <xacro:macro name="rear_wheel"
-                 params="lr_prefix lr_reflect">
-      <joint name="rear_${lr_prefix}_wheel_joint" type="continuous">
-        <origin xyz="${-1 * wheelbase / 2}
+                     0" rpy="0 0 0"/>
+				<parent link="base_footprint"/>
+				<child link="${lr_prefix}_steering_hinge"/>
+				<axis xyz="0 0 1"/>
+				<limit lower="${config['input_ranges']['steering']['min']}" upper="${config['input_ranges']['steering']['max']}" effort="10000000" velocity="1000000"/>
+			</joint>
+			<link name="${lr_prefix}_steering_hinge">
+				<inertial>
+					<origin xyz="0 0 0" rpy="0 0 0" />
+					<mass value="${steering_hinge_mass}"/>
+					<inertia ixx="0.04" ixy="0.0" ixz="0.0" iyy="0.04" iyz="0.0" izz="0.04" />
+				</inertial>
+			</link>
+			<joint name="front_${lr_prefix}_wheel_joint" type="continuous">
+				<origin xyz="0 0 0" rpy="0 0 0"/>
+				<parent link="${lr_prefix}_steering_hinge"/>
+				<child link="${lr_prefix}_front_wheel"/>
+				<axis xyz="0 1 0"/>
+				<limit lower="0" upper="0" effort="10000000" velocity="1000000"/>
+			</joint>
+			<xacro:wheel lr_prefix="${lr_prefix}" fr_prefix="front"/>
+		</xacro:macro>
+		<!-- Description of how a rear wheel is connected to the base_footprint -->
+		<xacro:macro name="rear_wheel" params="lr_prefix lr_reflect">
+			<joint name="rear_${lr_prefix}_wheel_joint" type="continuous">
+				<origin xyz="${-1 * wheelbase / 2}
                      ${lr_reflect * ((chassis_width - wheel_width) / 2)}
-                     0"
-                rpy="0 0 0"/>
-        <parent link="base_footprint"/>
-        <child link="${lr_prefix}_rear_wheel"/>
-        <axis xyz="0 1 0"/>
-        <limit lower="0" upper="0" effort="10000000" velocity="1000000"/>
-      </joint>
-      <xacro:wheel lr_prefix="${lr_prefix}" fr_prefix="rear"/>
-    </xacro:macro>
-    <!-- ************** -->
-    <!-- Add the wheels -->
-    <!-- ************** -->
-    <xacro:front_wheel lr_prefix="left" lr_reflect="1"/>
-    <xacro:front_wheel lr_prefix="right" lr_reflect="-1"/>
-    <xacro:rear_wheel lr_prefix="left" lr_reflect="1" />
-    <xacro:rear_wheel lr_prefix="right" lr_reflect="-1" />
-  </xacro:macro>
+                     0" rpy="0 0 0"/>
+				<parent link="base_footprint"/>
+				<child link="${lr_prefix}_rear_wheel"/>
+				<axis xyz="0 1 0"/>
+				<limit lower="0" upper="0" effort="10000000" velocity="1000000"/>
+			</joint>
+			<xacro:wheel lr_prefix="${lr_prefix}" fr_prefix="rear"/>
+		</xacro:macro>
+		<!-- ************** -->
+		<!-- Add the wheels -->
+		<!-- ************** -->
+		<xacro:front_wheel lr_prefix="left" lr_reflect="1"/>
+		<xacro:front_wheel lr_prefix="right" lr_reflect="-1"/>
+		<xacro:rear_wheel lr_prefix="left" lr_reflect="1" />
+		<xacro:rear_wheel lr_prefix="right" lr_reflect="-1" />
+	</xacro:macro>
 </robot>

Commit message: Fixed sensor placement

File: qutms_description/qev/qev.urdf.xacro (robot description, xacro)
@@ -1,5 +1,5 @@
 <?xml version="1.0"?>
 <robot xmlns:xacro="http://www.ros.org/wiki/xacro" name="qev">
-    <xacro:property name="M_PI" value="3.1415926535897931" />
+  <xacro:property name="M_PI" value="3.1415926535897931" />
     <!-- ***************** -->
     <!-- Config parameters -->
@@ -28,22 +28,24 @@
     <!-- ************** -->
     <!-- Chassis of the car -->
-    <xacro:car_base chassis_length="2.165" chassis_width="0.735" chassis_height="0.63"/>
+    <xacro:car_base chassis_length="2.165"
+                    chassis_width="0.735"
+                    chassis_height="0.63"/>
     <!-- Wheels -->
     <xacro:wheels chassis_width="2" wheelbase="2.0"/>
     <!-- GPS -->
-    <xacro:qev2_gps parent="base_footprint">
-        <origin xyz="0 0 0.71" rpy="0 0 0" />
+    <xacro:qev2_gps parent="base_footprint" >
+      <origin xyz="0 0 0.345" rpy="0 0 0" />
     </xacro:qev2_gps>
     <!-- IMU -->
-    <xacro:qev2_imu parent="base_footprint">
-        <origin xyz="0 0 0" rpy="0 0 ${M_PI/2}" />
+    <xacro:qev2_imu parent="base_footprint" >
+      <origin xyz="0 0 0" rpy="0 0 ${M_PI/2}" />
     </xacro:qev2_imu>
     <!-- LiDAR -->
     <xacro:qev2_horizon_lidar parent="base_footprint">
-        <origin xyz="1.1 0 0.1" rpy="0 0 0" />
+      <origin xyz="1.17 0 -0.24" rpy="0 0 0" />
     </xacro:qev2_horizon_lidar>
     <!-- Camera -->
     <xacro:qev2_zed_camera parent="base_footprint">
-        <origin xyz="-0.4 0 1.3" rpy="0 0 0" />
+      <origin xyz="-0.4 0 1.3" rpy="0 0 0" />
     </xacro:qev2_zed_camera>
 </robot>

File: qutms_description/urdf/sensors/qev2_zed_camera.urdf.xacro (robot description, xacro)
@@ -28,5 +28,5 @@
 			</collision>
 		</link>
-		<gazebo reference="${name}_base_link">
+		<gazebo reference="${name}_base_footprint">
 			<sensor type="multicamera" name="${name}">
 				<update_rate>30.0</update_rate>

Commit message: clean up sensor files

File: qutms_description/qev/qev.urdf.xacro (robot description, xacro)
@@ -1,5 +1,5 @@
 <?xml version="1.0"?>
 <robot xmlns:xacro="http://www.ros.org/wiki/xacro" name="qev">
-  <xacro:property name="M_PI" value="3.1415926535897931" />
+    <xacro:property name="M_PI" value="3.1415926535897931" />
     <!-- ***************** -->
     <!-- Config parameters -->
@@ -17,35 +17,33 @@
     <xacro:include filename="$(find qutms_description)/urdf/plugins.gazebo.xacro"/>
     <!-- GPS -->
-    <xacro:include filename="$(find qutms_description)/urdf/sensors/qev2_gps.urdf.xacro" />
+    <xacro:include filename="$(find qutms_description)/sensors/gps.urdf.xacro" />
     <!-- IMU -->
-    <xacro:include filename="$(find qutms_description)/urdf/sensors/qev2_imu.urdf.xacro" />
+    <xacro:include filename="$(find qutms_description)/sensors/imu.urdf.xacro" />
     <!-- LIDAR -->
-    <xacro:include filename="$(find qutms_description)/urdf/sensors/qev2_horizon_lidar.urdf.xacro"/>
+    <xacro:include filename="$(find qutms_description)/sensors/horizon_lidar.urdf.xacro"/>
     <!-- Camera -->
-    <xacro:include filename="$(find qutms_description)/urdf/sensors/qev2_zed_camera.urdf.xacro" />
+    <xacro:include filename="$(find qutms_description)/sensors/zed_camera.urdf.xacro" />
     <!-- ************** -->
     <!-- Robot Elements -->
     <!-- ************** -->
     <!-- Chassis of the car -->
-    <xacro:car_base chassis_length="2.165"
-                    chassis_width="0.735"
-                    chassis_height="0.63"/>
+    <xacro:car_base chassis_length="2.165" chassis_width="0.735" chassis_height="0.63"/>
     <!-- Wheels -->
     <xacro:wheels chassis_width="2" wheelbase="2.0"/>
     <!-- GPS -->
-    <xacro:qev2_gps parent="base_footprint" >
-      <origin xyz="0 0 0.345" rpy="0 0 0" />
-    </xacro:qev2_gps>
+    <xacro:gps parent="base_footprint">
+        <origin xyz="0 0 0.345" rpy="0 0 0" />
+    </xacro:gps>
     <!-- IMU -->
-    <xacro:qev2_imu parent="base_footprint" >
-      <origin xyz="0 0 0" rpy="0 0 ${M_PI/2}" />
-    </xacro:qev2_imu>
+    <xacro:imu parent="base_footprint">
+        <origin xyz="0 0 0" rpy="0 0 ${M_PI/2}" />
+    </xacro:imu>
     <!-- LiDAR -->
-    <xacro:qev2_horizon_lidar parent="base_footprint">
-      <origin xyz="1.17 0 -0.24" rpy="0 0 0" />
-    </xacro:qev2_horizon_lidar>
+    <xacro:horizon_lidar parent="base_footprint">
+        <origin xyz="1.17 0 -0.24" rpy="0 0 0" />
+    </xacro:horizon_lidar>
     <!-- Camera -->
-    <xacro:qev2_zed_camera parent="base_footprint">
-      <origin xyz="-0.4 0 1.3" rpy="0 0 0" />
-    </xacro:qev2_zed_camera>
+    <xacro:zed_camera parent="base_footprint">
+        <origin xyz="-0.4 0 1.3" rpy="0 0 0" />
+    </xacro:zed_camera>
 </robot>

File: qutms_description/sensors/gps.urdf.xacro (robot description, xacro)
@@ -1,5 +1,5 @@
 <?xml version="1.0"?>
 <robot xmlns:xacro="http://ros.org/wiki/xacro">
-	<xacro:macro name="qev2_gps" params="*origin parent:=base_footprint name:=gps topic_name:=gps/data update_rate:=30.0">
+	<xacro:macro name="gps" params="*origin parent:=base_footprint name:=gps topic_name:=gps/data update_rate:=30.0">
 		<!-- GPS Base Mount Joint -->
 		<joint name="${name}_base_mount_joint" type="fixed">
@@ -29,5 +29,5 @@
 		</link>
 		<gazebo>
-			<plugin name="gps_controller_${name}" filename="libhector_gazebo_ros_gps.so">
+			<plugin name="gps_plugin" filename="libhector_gazebo_ros_gps.so">
 				<robotNamespace>qev</robotNamespace>
 				<updateRate>30</updateRate>

File: qutms_description/sensors/horizon_lidar.urdf.xacro (robot description, xacro)
@@ -1,6 +1,6 @@
 <?xml version="1.0"?>
-<robot xmlns:xacro="http://ros.org/wiki/xacro" name="Horizon">
-    <xacro:property name="M_PI" value="3.1415926535897931" />
-    <xacro:macro name="qev2_horizon_lidar" params=" *origin parent:=base_footprint name:=horizon_lidar">
+<robot xmlns:xacro="http://ros.org/wiki/xacro">
+    <xacro:macro name="horizon_lidar" params=" *origin parent:=base_footprint name:=horizon_lidar">
+        <xacro:property name="M_PI" value="3.1415926535897931" />
         <joint name="${name}_base_mount_joint" type="fixed">
             <xacro:insert_block name="origin" />
@@ -57,5 +57,6 @@
                     </noise>
                 </ray>
-                <plugin name="qev2_lidar_plugin" filename="libhorizon_lidar_plugin.so">
+                <plugin name="lidar_plugin" filename="libhorizon_lidar_plugin.so">
+                    <robotNamespace>qev</robotNamespace>
                     <topicName>${name}/pointcloud</topicName>
                     <frameName>${name}_base_footprint</frameName>

File: qutms_description/sensors/imu.urdf.xacro (robot description, xacro)
@@ -1,5 +1,5 @@
 <?xml version="1.0"?>
 <robot xmlns:xacro="http://ros.org/wiki/xacro">
-	<xacro:macro name="qev2_imu" params="*origin parent:=base_footprint name:=imu topic_name:=imu/data update_rate:=30.0">
+	<xacro:macro name="imu" params="*origin parent:=base_footprint name:=imu topic_name:=imu/data update_rate:=30.0">
 		<!-- IMU Base Mount Joint -->
 		<joint name="${name}_base_mount_joint" type="fixed">
@@ -29,5 +29,5 @@
 		</link>
 		<gazebo>
-			<plugin name="imu_controller_${name}" filename="libhector_gazebo_ros_imu.so">
+			<plugin name="imu_plugin" filename="libhector_gazebo_ros_imu.so">
 				<robotNamespace>qev</robotNamespace>
 				<updateRate>${update_rate}</updateRate>

File: qutms_description/sensors/zed_camera.urdf.xacro (robot description, xacro)
@@ -1,5 +1,5 @@
 <?xml version="1.0"?>
 <robot xmlns:xacro="http://ros.org/wiki/xacro">
-	<xacro:macro name="qev2_zed_camera" params="*origin parent:=base_footprint name:=zed_camera">
+	<xacro:macro name="zed_camera" params="*origin parent:=base_footprint name:=zed_camera">
 		<!-- Camera Base Mount Joint -->
 		<joint name="${name}_base_mount_joint" type="fixed">
@@ -67,5 +67,6 @@
 					</noise>
 				</camera>
-				<plugin name="qev2_camera_plugin" filename="libgazebo_ros_multicamera.so">
+				<plugin name="camera_plugin" filename="libgazebo_ros_multicamera.so">
+					<robotNamespace>qev</robotNamespace>
 					<alwaysOn>true</alwaysOn>
 					<updateRate>0.0</updateRate>

Commit message: Changed camera placement

File: qutms_description/qev/qev.urdf.xacro (robot description, xacro)
@@ -45,5 +45,5 @@
     <!-- Camera -->
     <xacro:zed_camera parent="base_footprint">
-        <origin xyz="-0.4 0 1.3" rpy="0 0 0" />
+        <origin xyz="-0.4 0 0.9" rpy="0 0 0" />
     </xacro:zed_camera>
 </robot>
